File: pcb/hackpad.kicad_sch (KiCad schematic)
At the start: 47 parts, among them SW1 SW_Push, SW10 SW_Push, SW11 RotaryEncoder_Switch, SW2 SW_Push, SW3 SW_Push, SW4 SW_Push, SW5 SW_Push, SW6 SW_Push, SW7 SW_Push, SW8 SW_Push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

Commit message: Everything updated
Parts:
- removed C10, C6: C, Capacitor_SMD:C_0805_2012Metric, symbol Device:C
- removed D10, D5: 1N4148, Diode_THT:D_DO-35_SOD27_P7.62mm_Horizontal, symbol Diode:1N4148
- removed D18, D20: SK6812MINI, LED_SMD:LED_SK6812MINI_PLCC4_3.5x3.5mm_P1.75mm, symbol LED:SK6812MINI
- removed SW10, SW5: SW_Push, Kailh_PG1353_Hotswap:Kailh-PG1353-Hotswap-1U, symbol Switch:SW_Push
Connections:
- net Row 0: now also U1.6 (GPIO7/SCL); no longer U1.5 (GPIO6/SDA)
- net Row 1: now also U1.5 (GPIO6/SDA); no longer U1.6 (GPIO7/SCL)
- net at D19.3 (DIN): now also D17.1 (DOUT)
- net at D11.3 (DIN), R1.1: now also D14.1 (DOUT)
- net at D16.1 (DOUT): now also D13.3 (DIN)
- net at D15.1 (DOUT): now also D12.3 (DIN)
- net Col 4: no longer names the net of U1.10 (GPIO4/MISO)

Commit message: updated pcb final
Connections:
- net at D19.1 (DOUT): now also D14.3 (DIN); no longer D17.3 (DIN)
- net at D19.3 (DIN): now also D13.1 (DOUT); no longer D17.1 (DOUT)
- net at D11.1 (DOUT): now also D12.3 (DIN); no longer D14.3 (DIN)
- net at D11.3 (DIN), R1.1: now also D17.1 (DOUT); no longer D14.1 (DOUT)
- net at D16.1 (DOUT): now also D17.3 (DIN); no longer D13.3 (DIN)
- net at D16.3 (DIN): now also D15.1 (DOUT); no longer D13.1 (DOUT)
- net at D15.3 (DIN): now also D14.1 (DOUT); no longer D12.1 (DOUT)
- new net: D12.1 (DOUT), D13.3 (DIN)
Other:
- moved on the sheet: D1, D2, D3, D4, D6, D7, D8, D9, H1, H2, H3, H4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
